File: Q17_2final/Q17_2final.kicad_pcb (KiCad board)
At the start: 2 copper layers, 174.7 x 58.3 mm, 97 parts, among them J1 Input, J2 Screw_Terminal_01x02, J3 Screw_Terminal_01x03, Q1 IRF610, Q10 2SA970, Q11 BS250, Q12 2SC2240, Q13 IRF610, Q14 IRF9610, Q15 FQA46N15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

Commit message: Add files via upload
Parts:
- C10: value 47pF -> 47p
- C11, C19, C26, C27, C4, C5, C8, C9: value 100nF -> 100n
- C17: value 100nF FKP -> 100nF FKP
- C20, C21: value 2200uF/63V -> 4700uF/63V
- C22: value 220uF -> 220uF/6.3V
- R10, R13: value 10R -> 10
- R11, R12: value 47R/1W -> 47/1W
- R14, R15, R22, R33: value 330R -> 330
- R3: value 150R -> 150
- R7, R9: value 100R -> 100
- R8: value 120R -> 120
- moved R17 4.31 mm to (74.0, 106.1)
- moved R23 4.30 mm to (78.3, 106.1)
Routing:
- net Net-(J2-Pad2): track 96.3 -> 91.9 mm, vias 6 -> 4
- net Net-(C2-Pad1): track 10.8 -> 9.61 mm
- net Net-(Q8-Pad1): track 17.9 -> 16.8 mm
- net Net-(L1-Pad2): track 144.1 -> 143.4 mm
- added copper zone on F.Cu, net GNDPWR
Other:
- board text added: "GND"
- board text added: "Q17 PCB ver. 2.5 by Tiberiu Vicol"
- board text added: "QUAD405 Audiophile"
- board text added: "bipolar"
- board text added: "mica"
- board text removed: "QUAD405 Audiophile by Tiberiu Vicol"
- board text removed: "version 2.1"

Commit message: Add files via upload
Parts:
- removed the ? at (61.3, 102.7)
- C12, C18: value 100nF -> 100n
- C13: value 220uF/63V -> 220u/63V
- C17: value 100nF FKP -> 100n
- C2: value 220uF -> 220uF/16V
- C20, C21: value 4700uF/63V -> min. 2200u/63V
- C22: value 220uF/6.3V -> 2 X 220u/16V
- C3: value 100uF/25V -> 100u/25V
- C6: value 100uF/16V -> 100u/16V
- C7: value 1uF MKP -> 1u MKP
- R10, R13, R29, R30, R5: value 10 -> 10R
- R11, R12: value 47/1W -> 47R/1W
- R14, R15, R22, R33: value 330 -> 330R
- R2, R21: value 5k6/1W -> 10k
- R23: value 8K2 -> 8k2
- R3: value 150 -> 150R
- R32: value 10 -> 0R
- R34, R35, R36, R37: value 0R1 -> 0R1/2W
- R4, R7, R9: value 100 -> 100R
- R6: value 100/0.5W -> 100R
- R8: value 120 -> 120R
- moved ? 2.23 mm to (61.3, 99.4)
- moved ? 2.23 mm to (61.3, 91.9)
- moved C7 2.23 mm to (61.3, 76.9)
Connections:
- U1 pad 1: (no net) -> unconnected-(U1-Pad1)
- U1 pad 5: (no net) -> unconnected-(U1-Pad5)
- U1 pad 8: (no net) -> unconnected-(U1-Pad8)
Routing:
- net Net-(C7-Pad2): track 25.8 -> 23.0 mm
- net Net-(C7-Pad1): track 47.2 -> 46.4 mm
- net GNDPWR: vias 0 -> 22
- net GND: vias 0 -> 31
Other:
- board text added: "FKP"
- board text added: "Q17 PCB ver. 2.7 by Tiberiu Vicol"
- board text removed: "Q17 PCB ver. 2.5 by Tiberiu Vicol"

Commit message: KiCad files for Q17 2 pair pcb ver.2.8
Other:
- board text added: "Q17 PCB ver.2.8 by Tiberiu Vicol"
- board text removed: "Q17 PCB ver. 2.7 by Tiberiu Vicol"
Changed lines of the file:
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@@
   (title_block
     (title "QUAD405 Reborn")
-    (date "2021-04-15")
-    (rev "17")
+    (date "2022-12-11")
+    (rev "2.7")
   )
   (layers
@@
       (effects (font (size 1.3 1.3) (thickness 0.2)))
     )
-    (fp_text user "cap. outer foil" (at 0 3.14 90 unlocked) (layer "F.SilkS")
+    (fp_text user "outer foil" (at 0 3.14 90 unlocked) (layer "F.SilkS")
       (effects (font (size 1 1) (thickness 0.15)))
     )
@@
     (fp_line (start -1.45 -6.75) (end -1.45 6.75) (layer "F.SilkS") (width 0.05))
     (fp_line (start 0.78 -2.6) (end 2.58 -2.6) (layer "F.SilkS") (width 0.25))
-    (pad "1" thru_hole oval (at 0 0 270) (size 2.4 2.4) (drill 1.2) (layers *.Cu *.Mask)
+    (pad "1" thru_hole circle (at 0 0 270) (size 2.7 2.7) (drill 1.5) (layers *.Cu *.Mask)
       (net 35 "Net-(C7-Pad1)") (pintype "passive"))
-    (pad "2" thru_hole roundrect (at 26 0 270) (size 2.4 2.4) (drill 1.2) (layers *.Cu *.Mask) (roundrect_rratio 0.25)
+    (pad "2" thru_hole roundrect (at 26 0 270) (size 2.7 2.7) (drill 1.5) (layers *.Cu *.Mask) (roundrect_rratio 0.25)
       (net 7 "Net-(C7-Pad2)") (pintype "passive"))
     (model "${KICAD6_3DMODEL_DIR}/Capacitor_THT.3dshapes/CP_Axial_L20.0mm_D13.0mm_P26.00mm_Horizontal.wrl"
@@
     (fp_line (start -1.5 -5.5) (end -1.5 5.5) (layer "F.Fab") (width 0.1))
     (fp_line (start 16.5 -5.5) (end -1.5 -5.5) (layer "F.Fab") (width 0.1))
-    (pad "1" thru_hole circle locked (at 0 0 270) (size 2.4 2.4) (drill 1.2) (layers *.Cu *.Mask)
+    (pad "1" thru_hole circle locked (at 0 0 270) (size 2.7 2.7) (drill 1.5) (layers *.Cu *.Mask)
       (net 19 "Net-(C17-Pad1)") (pintype "passive"))
     (pad "2" thru_hole circle locked (at 10 0 270) (size 2.4 2.4) (drill 1.2) (layers *.Cu *.Mask)
       (net 13 "GNDPWR") (pintype "passive"))
-    (pad "2" thru_hole circle locked (at 15 0 270) (size 2.4 2.4) (drill 1.2) (layers *.Cu *.Mask)
+    (pad "2" thru_hole circle locked (at 15 0 270) (size 2.7 2.7) (drill 1.5) (layers *.Cu *.Mask)
       (net 13 "GNDPWR") (pintype "passive"))
     (model "${KICAD6_3DMODEL_DIR}/Capacitor_THT.3dshapes/C_Rect_L18.0mm_W11.0mm_P15.00mm_FKS3_FKP3.wrl"
@@
     (effects (font (size 1.4 1.4) (thickness 0.2)))
   )
-  (gr_text "Q17 PCB ver. 2.7\nby Tiberiu Vicol" (at 216.26 105.33) (layer "F.SilkS")
+  (gr_text "Q17 PCB ver.2.8\nby Tiberiu Vicol" (at 215.51 105.33) (layer "F.SilkS")
     (effects (font (size 1.1 1.1) (thickness 0.2)))
   )
@@
     (effects (font (size 1 1) (thickness 0.15)))
   )
-  (dimension (type aligned) (layer "F.Cu")
+  (dimension (type aligned) (layer "User.1")
     (pts (xy 208.11 37.86) (xy 208.26 142.67))
     (height -36.20959)
-    (gr_text "104.8101 mm" (at 246.194551 90.210602 270.0819994) (layer "F.Cu")
+    (gr_text "104.8101 mm" (at 246.194551 90.210602 270.0819994) (layer "User.1")
       (effects (font (size 1.5 1.5) (thickness 0.3)))
     )
@@
     (style (thickness 0.2) (arrow_length 1.27) (text_position_mode 0) (extension_height 0.58642) (extension_offset 0.5) keep_text_aligned)
   )
-  (dimension (type aligned) (layer "Margin")
-    (pts (xy 175.72 77.87) (xy 198.02 77.84))
+  (dimension (type aligned) (layer "User.1")
+    (pts (xy 175.72 60.650417) (xy 198.02 60.620417))
     (height -22.692374)
-    (gr_text "22.3000 mm" (at 186.837925 54.012648 0.07707947751) (layer "Margin")
+    (gr_text "22.3000 mm" (at 186.837925 36.793065 0.07707947751) (layer "User.1")
       (effects (font (size 1 1) (thickness 0.15)))
     )

Commit message: Add files via upload
Parts:
- C6: value 100u/16V -> 100u/25V
Other:
- board text added: "Q17 PCB ver.2.9 by VAT"
- board text removed: "Q17 PCB ver.2.8 by Tiberiu Vicol"
