File: Q17_2final/Q17_2final.kicad_sch (KiCad schematic)
At the start: 91 parts, among them J1 Input, J2 Screw_Terminal_01x02, J3 Screw_Terminal_01x03, Q1 IRF610, Q10 2SA970, Q11 BS250, Q12 2SC2240 / AC181, Q13 IRF610, Q14 IRF9610, Q15 FQA46N15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

Commit message: Add files via upload
Parts:
- R2: value 5k6/1W -> 10K/1W
- R21: value 5k6/1W -> 10k/1W
- R32: value 10 -> 0
Changed lines of the file:
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@@
       (effects (font (size 1.27 1.27)) (justify left))
     )
-    (property "Value" "5k6/1W" (id 1) (at 82.042 114.421 0)
+    (property "Value" "10k/1W" (id 1) (at 82.042 114.421 0)
       (effects (font (size 1.27 1.27)) (justify left))
     )
@@
       (effects (font (size 1.27 1.27)) (justify left))
     )
-    (property "Value" "5k6/1W" (id 1) (at 82.042 53.473 0)
+    (property "Value" "10K/1W" (id 1) (at 82.042 53.473 0)
       (effects (font (size 1.27 1.27)) (justify left))
     )
@@
       (effects (font (size 1.27 1.27)) (justify left))
     )
-    (property "Value" "10" (id 1) (at 268.611 147.32 0)
+    (property "Value" "0" (id 1) (at 268.611 147.32 0)
       (effects (font (size 1.27 1.27)) (justify left))
     )
@@
     )
     (path "/66629faf-a191-4328-8001-bb82d5d2442f"
-      (reference "R2") (unit 1) (value "5k6/1W") (footprint "Resistor_THT:R_Axial_DIN0207_L6.3mm_D2.5mm_P10.16mm_Horizontal")
+      (reference "R2") (unit 1) (value "10K/1W") (footprint "Resistor_THT:R_Axial_DIN0207_L6.3mm_D2.5mm_P10.16mm_Horizontal")
     )
     (path "/86507d1a-5f15-441f-9633-93c496bb3e70"
@@
     )
     (path "/1b488199-e780-425b-bf65-6607168f9f34"
-      (reference "R21") (unit 1) (value "5k6/1W") (footprint "Resistor_THT:R_Axial_DIN0207_L6.3mm_D2.5mm_P10.16mm_Horizontal")
+      (reference "R21") (unit 1) (value "10k/1W") (footprint "Resistor_THT:R_Axial_DIN0207_L6.3mm_D2.5mm_P10.16mm_Horizontal")
     )
     (path "/3a342a55-d71d-42e5-8f4a-082ea0da699a"
@@
     )
     (path "/f62732fe-8027-4c0c-a9a9-204da2bf2115"
-      (reference "R32") (unit 1) (value "10") (footprint "Resistor_THT:R_Axial_DIN0207_L6.3mm_D2.5mm_P10.16mm_Horizontal")
+      (reference "R32") (unit 1) (value "0") (footprint "Resistor_THT:R_Axial_DIN0207_L6.3mm_D2.5mm_P10.16mm_Horizontal")
     )
     (path "/f2b0d193-7888-47c1-885e-3ee6da907697"

Commit message: Add files via upload
Parts:
- C11, C12, C18, C19, C26, C27, C4, C5, C8, C9: Spice_Model 100n -> (none); Spice_Netlist_Enabled Y -> (none); Spice_Primitive C -> (none)
